File: Master_Glove/Master_Glove.kicad_sch (KiCad schematic)
At the start: 0 parts

Commit message: Excel calculation and creation of division in project
Small push with All pages created with naming following how tasks were seperated before placing components
Other:
- added sheet Capacitor Charge Discharge (Capacitor_Charge_Discharge.kicad_sch)
- added sheet Conversion and display (Display.kicad_sch)
- added sheet Emitter (Emitter.kicad_sch)
- added sheet Math (Math.kicad_sch)
- added sheet Power (Power.kicad_sch)
- added sheet Receptor (Receptor.kicad_sch)
- company: (none) -> C3I
- title: (none) -> Glove PCB
