File: Master_Glove/Power.kicad_sch (KiCad schematic)
At the start: 0 parts

Commit message: Power
Parts:
- added BT1: 1.2V, EasyEda2Kicad:CONN-TH_B2B-PH-K-S, symbol Device:Battery_Cell
- added C17, C18: 10u, symbol Device:C_Small
- added C19: 0.47u, symbol Device:C_Small
- added F1: Polyfuse_Small, Resistor_SMD:R_0603_1608Metric_Pad0.98x0.95mm_HandSolder, symbol Device:Polyfuse_Small
- added L1: 4.7u, symbol Device:L_Small
- added Q1: PMOS, EasyEda2Kicad:SOT-23-3_L2.9-W1.3-P1.90-LS2.4-BR, symbol Simulation_SPICE:PMOS
- added R37: R_Small_US, Resistor_SMD:R_0603_1608Metric_Pad0.98x0.95mm_HandSolder, symbol Device:R_Small_US
- added R38: 1.74M, symbol Device:R_Small_US
- added R39: 180k, symbol Device:R_Small_US
- added R40: 1M, symbol Device:R_Small_US
- added R41: 3.16M, symbol Device:R_Small_US
- added SW2: SW_SPST, symbol Switch:SW_SPST
- added U13: TLV61220DBVR, Library:SOT-23-6_L2.9-W1.6-P0.95-LS2.8-BR, symbol Library:TLV61220DBVR
- added U14: TLV709A50DBVR, Library:TSOT-23-5_L2.9-W1.6-P0.95-LS2.8-BR, symbol Library:TLV709A50DBVR
Connections:
- new net: L1.2, U13.1 (SW)
- new net: R38.2, R39.1, U13.4 (FB)
- new net: BT1.1 (+), SW2.1 (A)
- new net: F1.1, SW2.2 (B)
- new net: F1.2, Q1.1 (D)
- new net: Q1.3 (S), R37.1
- new net: R40.2, R41.1, U14.4 (FB)
- new net 5.3V: C18.1, R38.1, U13.5 (VOUT), U14.1 (IN)
- new net GND: BT1.2 (-), C17.2, C18.2, C19.2, Q1.2 (G), R39.2, R41.2, U13.2 (GND), U14.2 (GND), U14.3 (NC)
- new net VBatt: C17.1, L1.1, R37.2, U13.3 (EN), U13.6 (VBAT)
- new net VCC: C19.1, R40.1, U14.5 (OUT)

Commit message: Modifications according to reccomendation
Changed Vcc to +5V
Subbed MIC1551 to MIC 1553
Added debounce on button
Fixed other small bugs
Connections:
- net VCC renamed +5V
Changed lines of the file:
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@@
 			)
 		)
-		(property "Value" "VCC"
+		(property "Value" "+5V"
 			(at 167.64 29.464 0)
 			(effects

Commit message: Adding footprints
Changed lines of the file:
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@@
+	(wire
+		(pts
+			(xy 167.64 31.75) (xy 167.64 33.02)
+		)
+		(stroke
+			(width 0)
+			(type default)
+		)
+	)
 	(wire
 		(pts
@@
 	(symbol
 		(lib_id "power:+3V8")
-		(at 167.64 33.02 0)
+		(at 167.64 31.75 0)
 		(unit 1)
 		(exclude_from_sim no)
@@
 		(dnp no)
 		(property "Reference" "#PWR076"
-			(at 167.64 36.83 0)
+			(at 167.64 35.56 0)
 			(effects
 				(font
@@
 		)
 		(property "Value" "+5V"
-			(at 167.64 29.464 0)
-			(effects
-				(font
-					(size 1.27 1.27)
-				)
-			)
-		)
-		(property "Footprint" ""
-			(at 167.64 33.02 0)
+			(at 167.64 28.194 0)
+			(effects
+				(font
+					(size 1.27 1.27)
+				)
+			)
+		)
+		(property "Footprint" ""
+			(at 167.64 31.75 0)
 			(effects
 				(font
@@
 		)
 		(property "Datasheet" ""
-			(at 167.64 33.02 0)
+			(at 167.64 31.75 0)
 			(effects
 				(font
@@
 		)
 		(property "Description" "Power symbol creates a global label with name \"+3V8\""
-			(at 167.64 33.02 0)
-			(effects
-				(font
+			(at 167.64 31.75 0)
+			(effects
+				(font
