File: Master_Glove/Receptor.kicad_sch (KiCad schematic)
At the start: 0 parts

Commit message: Power
Parts:
- added LS1: Receptor, symbol Device:Speaker_Ultrasound
- added U15: LMH6609MA, Package_SO:SOIC-8_3.9x4.9mm_P1.27mm, symbol Amplifier_Operational:LMH6609MA
Connections:
- new net: LS1.1, U15.3 (+)
- new net 5V: U15.7 (V+)
- new net GND: LS1.2, U15.4 (V-)
- new net SIGNAL_ISOLE: U15.2 (-), U15.6

Commit message: added footprints
Parts:
- LS1: footprint (none) -> LCSC:SENSOR-TH_GU10XXC-40TR
Changed lines of the file:
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@@
 			)
 		)
-		(property "Footprint" ""
+		(property "Footprint" "LCSC:SENSOR-TH_GU10XXC-40TR"
 			(at 27.559 59.69 0)
 			(effects
@@
 			)
 		)
-		(property "Datasheet" "~"
+		(property "Datasheet" "https://www.lcsc.com/product-detail/C242178.html"
 			(at 27.559 59.69 0)
 			(effects
